File: voltage_regulator_3_3V.kicad_pcb (KiCad board)
At the start: 2 copper layers, 14 x 33.5 mm, 13 parts, among them P1 USB_C_Plug_USB2.0, P2 USB_C_Plug_USB2.0, U1 AP2112K-3.3

Commit message: schematic and pcb update
Parts:
- removed P2: USB_C_Plug_USB2.0, SMD_TYPE-C-006:USB-C-SMD_USB-TYPE-C-006_USB-TYPE-C-006_C2927026
- added G***: LOGO, _Logo:logo_6mm, B.Cu at (134.2, 79.5)
- added J1: Screw_Terminal_01x02, TerminalBlock:TerminalBlock_bornier-2_P5.08mm, F.Cu at (140.5, 72.4)
- moved P1 0.64 mm to (138.0, 97.1)
Routing:
- net /3.3V: track 19.6 -> 23.8 mm
- net GND: track 0.00 -> 1.40 mm, vias 27 -> 29
- net /5V: track 16.2 -> 17.0 mm
Other:
- board text added: "3.3V"
- board text added: "5V"
- board text added: "5V to 3.3V voltage regulator"
