File: voltage_regulator_3_3V.kicad_sch (KiCad schematic)
At the start: 13 parts, among them P1 USB_C_Plug_USB2.0, P2 USB_C_Plug_USB2.0, U1 AP2112K-3.3

Commit message: schematic and pcb update
Parts:
- removed P2: USB_C_Plug_USB2.0, SMD_TYPE-C-006:USB-C-SMD_USB-TYPE-C-006_USB-TYPE-C-006_C2927026, symbol Connector:USB_C_Plug_USB2.0
- added J1: Screw_Terminal_01x02, TerminalBlock:TerminalBlock_bornier-2_P5.08mm, symbol Connector:Screw_Terminal_01x02
Connections:
- net 3.3V: now also J1.1 (Pin_1)
- net GND: now also J1.2 (Pin_2)
- no-connect marks 8 -> 4
Changed lines of the file:
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@@
-	)
-	(junction
-		(at 213.36 114.3)
-		(diameter 0)
-		(color 0 0 0 0)
 	)
 	(junction
@@
 	)
 	(no_connect
-		(at 198.12 81.28)
-	)
-	(no_connect
-		(at 198.12 86.36)
-	)
-	(no_connect
-		(at 198.12 91.44)
-	)
-	(no_connect
 		(at 86.36 91.44)
 	)
@@
 		(at 86.36 81.28)
 	)
-	(no_connect
-		(at 198.12 78.74)
-	)
 	(wire
 		(pts
@@
 	(wire
 		(pts
-			(xy 194.31 114.3) (xy 213.36 114.3)
-		)
-		(stroke
-			(width 0)
-			(type default)
-		)
-	)
-	(wire
-		(pts
 			(xy 93.98 73.66) (xy 93.98 78.74)
 		)
@@
 	(wire
 		(pts
+			(xy 198.12 76.2) (xy 198.12 114.3)
+		)
+		(stroke
+			(width 0)
+			(type default)
+		)
+	)
+	(wire
+		(pts
 			(xy 144.78 114.3) (xy 152.4 114.3)
 		)
@@
 	(wire
 		(pts
+			(xy 198.12 114.3) (xy 194.31 114.3)
+		)
+		(stroke
+			(width 0)
+			(type default)
+		)
+	)
+	(wire
+		(pts
 			(xy 71.12 114.3) (xy 71.12 111.76)
 		)
@@
 	(wire
 		(pts
-			(xy 220.98 114.3) (xy 220.98 111.76)
-		)
-		(stroke
-			(width 0)
-			(type default)
-		)
-	)
-	(wire
-		(pts
 			(xy 71.12 114.3) (xy 93.98 114.3)
 		)
@@
 	(wire
 		(pts
-			(xy 213.36 111.76) (xy 213.36 114.3)
-		)
-		(stroke
-			(width 0)
-			(type default)
-		)
-	)
-	(wire
-		(pts
 			(xy 144.78 83.82) (xy 144.78 114.3)
 		)
@@
 		(pts
 			(xy 114.935 73.66) (xy 114.935 83.82)
-		)
-		(stroke
-			(width 0)
-			(type default)
-		)
-	)
-	(wire
-		(pts
-			(xy 213.36 114.3) (xy 220.98 114.3)
 		)
 		(stroke
@@
 	)
 	(symbol
-		(lib_id "Connector:USB_C_Plug_USB2.0")
-		(at 213.36 88.9 0)
-		(mirror y)
+		(lib_id "Connector:Screw_Terminal_01x02")
+		(at 203.2 73.66 0)
 		(unit 1)
 		(body_style 1)
@@
 		(in_pos_files yes)
 		(dnp no)
-		(property "Reference" "P2"
-			(at 224.79 90.1701 0)
-			(show_name no)
-			(do_not_autoplace no)
-			(effects
-				(font
-					(size 1.27 1.27)
-				)
-				(justify right)
-			)
-		)
-		(property "Value" "USB_C_Plug_USB2.0"
-			(at 224.79 87.6301 0)
-			(show_name no)
-			(do_not_autoplace no)
-			(effects
-				(font
-					(size 1.27 1.27)
-				)
-				(justify right)
-			)
-		)
-		(property "Footprint" "SMD_TYPE-C-006:USB-C-SMD_USB-TYPE-C-006_USB-TYPE-C-006_C2927026"
-			(at 209.55 88.9 0)
-			(hide yes)
-			(show_name no)
-			(do_not_autoplace no)
-			(effects
-				(font
-					(size 1.27 1.27)
-				)
-			)
-		)
-		(property "Datasheet" "https://www.usb.org/sites/default/files/documents/usb_type-c.zip"
-			(at 209.55 88.9 0)
-			(hide yes)
-			(show_name no)
-			(do_not_autoplace no)
-			(effects
-				(font
-					(size 1.27 1.27)
-				)
-			)
-		)
-		(property "Description" "USB 2.0-only Type-C Plug connector"
-			(at 213.36 88.9 0)
-			(hide yes)
-			(show_name no)
-			(do_not_autoplace no)
-			(effects
-				(font
-					(size 1.27 1.27)
-				)
-			)
-		)
-		(pin "B4"
-		)
-		(pin "A12"
-		)
-		(pin "B12"
-		)
-		(pin "B9"
-		)
-		(pin "B1"
-		)
-		(pin "A9"
-		)
-		(pin "SH"
-		)
-		(pin "B5"
-		)
-		(pin "A4"
-		)
-		(pin "A7"
-		)
-		(pin "A5"
-		)
-		(pin "A6"
-		)
-		(pin "A1"
+		(fields_autoplaced yes)
+		(property "Reference" "J1"
+			(at 205.74 73.6599 0)
+			(show_name no)
+			(do_not_autoplace no)
+			(effects
+				(font
+					(size 1.27 1.27)
+				)
+				(justify left)
+			)
+		)
+		(property "Value" "Screw_Terminal_01x02"
+			(at 205.74 76.1999 0)
+			(show_name no)
+			(do_not_autoplace no)
+			(effects
+				(font
+					(size 1.27 1.27)
+				)
+				(justify left)
+			)
+		)
+		(property "Footprint" "TerminalBlock:TerminalBlock_bornier-2_P5.08mm"
+			(at 203.2 73.66 0)
+			(hide yes)
+			(show_name no)
+			(do_not_autoplace no)
+			(effects
+				(font
+					(size 1.27 1.27)
+				)
+			)
+		)
+		(property "Datasheet" ""
+			(at 203.2 73.66 0)
+			(hide yes)
+			(show_name no)
+			(do_not_autoplace no)
+			(effects
+				(font
+					(size 1.27 1.27)
+				)
+			)
+		)
+		(property "Description" "Generic screw terminal, single row, 01x02, script generated (kicad-library-utils/schlib/autogen/connector/)"
+			(at 203.2 73.66 0)
+			(hide yes)
+			(show_name no)
+			(do_not_autoplace no)
+			(effects
+				(font
+					(size 1.27 1.27)
+				)
+			)
+		)
+		(pin "1"
+		)
+		(pin "2"
 		)
 		(instances
 			(project "voltage_regulator_3_3V"
 				(path "/f388d50b-5132-4741-9f78-ed93b89a92e2"
-					(reference "P2")
+					(reference "J1")
 					(unit 1)
 				)
